File: schematics/tms9981/bionic-tms9981-ldo.kicad_sch (KiCad schematic)
At the start: 11 parts, among them J1 Bionic-P135, J2 Bionic-P245, U1 TMS9981, U2 11AA010-I/TT, U3 LM78L12

Commit message: [TMS9981] Rename LDO version
Other:
- title: BionicTMS9981 -> BionicTMS9981 LDO
Changed lines of the file:
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@@
 	(paper "A4")
 	(title_block
-		(title "BionicTMS9981")
+		(title "BionicTMS9981 LDO")
 		(date "2024-12-28")
 		(rev "2")
