File: schematics/f3850/bionic-f3850-ldo.kicad_pcb (KiCad board)
At the start: 2 copper layers, 25.4 x 68.6 mm, 11 parts, among them J1 Bionic-P135, J2 Bionic-P245, U1 F3850, U2 11AA010-I/TT, U3 LM78L12

Commit message: [F3850] Rename LDO version
Other:
- rule pad_to_mask_clearance: 0.051 -> 0
Changed lines of the file:
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@@
 	(paper "A4")
 	(title_block
-		(title "BionicF3850")
+		(title "BionicF3850 LDO")
 		(date "2024-12-10")
 		(rev "5")
@@
 			(dielectric_constraints no)
 		)
-		(pad_to_mask_clearance 0.051)
-		(solder_mask_min_width 0.25)
+		(pad_to_mask_clearance 0)
 		(allow_soldermask_bridges_in_footprints no)
 		(aux_axis_origin 101 70)
@@
 			(drillshape 0)
 			(scaleselection 1)
-			(outputdirectory "gerber/")
+			(outputdirectory "gerber-ldo/")
 		)
 	)
@@
 			)
 		)
+		(model "${KIPRJMOD}/0-LocalLibrary/LED_CSL1901UW1_ROM.step"
+			(offset
+				(xyz 0 0 0)
+			)
+			(scale
+				(xyz 1 1 1)
+			)
+			(rotate
+				(xyz 0 0 0)
+			)
+		)
