File: schematics/f3850/dcdc+12v.kicad_sch (KiCad schematic)
At the start: 8 parts, among them U1 NJW4132

Commit message: [F3850] Cleanup schematics
Remove LDO version
Parts:
- C2: footprint Capacitor_SMD:C_1210_3225Metric_Pad1.33x2.70mm_HandSolder -> Capacitor_SMD:C_0603_1608Metric_Pad1.08x0.95mm_HandSolder
Changed lines of the file:
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@@
 			)
 		)
-		(property "Footprint" "Capacitor_SMD:C_1210_3225Metric_Pad1.33x2.70mm_HandSolder"
+		(property "Footprint" "Capacitor_SMD:C_0603_1608Metric_Pad1.08x0.95mm_HandSolder"
 			(at 101.6 68.58 0)
 			(effects
