File: schematics/z8002/bionic-z8002.kicad_sch (KiCad schematic)
At the start: 6 parts, among them J1 Bionic-P135, J2 Bionic-P245, U1 Z8002, U2 74HCT126, U3 11AA010-I/TO

Commit message: [WIP] [Z8002] Update schematics
Parts:
- removed C1: 0.1u, Capacitor_THT:C_Disc_D3.4mm_W2.1mm_P2.50mm, symbol Device:C_Small
- removed J1: Bionic-P135, connector:Bionic-P135_Vertical, symbol 0-LocalLibrary:Bionic-P135
- removed J2: Bionic-P245, connector:Bionic-P245_Vertical, symbol 0-LocalLibrary:Bionic-P245
- removed U1: Z8002, Package_DIP:DIP-40_W15.24mm, symbol 0-LocalLibrary:Z8002
- removed U2: 74HCT126, Package_DIP:DIP-14_W7.62mm, symbol 0-LocalLibrary:74HCT126
- removed U3: 11AA010-I/TO, TO-92_MC_MCH, symbol 0-LocalLibrary:11AA010-I_TO
- added D1: CSL1901UW1, rhom:LED_CSL1901UW1_ROM-M, symbol rhom:CSL1901UW1
- added J1: Bionic-P135, bionic:Bionic-P135_Vertical, symbol bionic:Bionic-P135
- added J2: Bionic-P245, bionic:Bionic-P245_Vertical, symbol bionic:Bionic-P245
- added U1: Z8002, bionic:DIP-40_W15.24mm_Socket, symbol cpu:Z8002
- added U2: 11AA010-I/TT, microchip:SOT-23_MC_MCH-M, symbol microchip:11AA010-I_TT
Connections:
- no-connect marks 7 -> 0
