File: schematics/z180/bionic-z180vsc.kicad_sch (KiCad schematic)
At the start: 11 parts, among them J1 Bionic-P135, J2 Bionic-P245, U1 Z80180, U2 11AA010-I/TT, U3 74AHCT157

Commit message: [Z180] Rename PLCC package project
Other:
- title: BionicZ180 -> BionicZ180VSC
Changed lines of the file:
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@@
 	(paper "A4")
 	(title_block
-		(title "BionicZ180")
-		(date "2025-10-12")
-		(rev "1")
+		(title "BionicZ180VSC")
+		(date "2025-11-17")
+		(rev "2")
 		(company "Tadashi G. Takaoka")
 	)
