File: schematics/p8051/bionic-p8051.kicad_sch (KiCad schematic)
At the start: 10 parts, among them J1 Bionic-P135, J2 Bionic-P245, U1 P8051AH, U2 11AA010-I/TT

Commit message: [i8051] Add automation config
Fix the samples' 16-bit division.
Connections:
- net P54: now also J2.29 (P54), U1.15 (P3.5); no longer J2.28 (P55), U1.14 (P3.4)
- net P55: now also J2.28 (P55), U1.14 (P3.4); no longer J2.29 (P54), U1.15 (P3.5)
