File: schematics/tms370cx5x/bionic-tms370cx5x.kicad_pcb (KiCad board)
At the start: 2 copper layers, 31.7 x 68.6 mm, 11 parts, among them J1 Bionic-P135, J2 Bionic-P245, U1 TMS370Cx5x, U2 11AA010-I/TT

Commit message: [tms370] Add automation config
Fix the samples' 16-bit division and resuming after an oscillator fault.
Connections:
- U1 pad 35: unconnected-(U1-VSS_{3}-Pad35) -> GND
- U1 pad 9: unconnected-(U1-VSS_{1}-Pad9) -> GND
Other:
- board text added: "Rev. 4"
- board text removed: "Rev. 3"
Changed lines of the file:
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@@
 	(title_block
 		(title "BionicTMS370Cx5x")
-		(date "2026-02-01")
-		(rev "3")
+		(date "2026-10-02")
+		(rev "4")
 		(company "Tadashi G. Takaoka")
 	)
@@
 	(net 64 "unconnected-(U1-SPISOMI-Pad49)")
 	(net 65 "unconnected-(U1-AN5-Pad41)")
-	(net 66 "unconnected-(U1-VSS_{3}-Pad35)")
-	(net 67 "unconnected-(U1-VSS_{1}-Pad9)")
 	(footprint "rhom:LED_CSL1901UW1_ROM-M"
 		(layer "F.Cu")
@@
 			(size 0.7 1.91)
 			(layers "F.Cu" "F.Mask" "F.Paste")
-			(net 67 "unconnected-(U1-VSS_{1}-Pad9)")
+			(net 2 "GND")
 			(pinfunction "VSS_{1}")
 			(pintype "power_in")
@@
 			(size 0.7 1.91)
 			(layers "F.Cu" "F.Mask" "F.Paste")
-			(net 66 "unconnected-(U1-VSS_{3}-Pad35)")
+			(net 2 "GND")
 			(pinfunction "VSS_{3}")
 			(pintype "power_in")
@@
 		)
 	)
-	(gr_arc
-		(start 99.095 138.58)
-		(mid 98.196974 138.208026)
+	(gr_line
+		(start 97.825 71.27)
 		(end 97.825 137.31)
 		(stroke
@@
 		(layer "Edge.Cuts")
 	)
-	(gr_line
-		(start 128.305 70)
+	(gr_arc
+		(start 97.825 71.27)
+		(mid 98.196974 70.371974)
 		(end 99.095 70)
 		(stroke
@@
 	)
 	(gr_arc
-		(start 97.825 71.27)
-		(mid 98.196974 70.371974)
-		(end 99.095 70)
+		(start 99.095 138.58)
+		(mid 98.196974 138.208026)
+		(end 97.825 137.31)
 		(stroke
 			(width 0.15)
@@
 		(layer "Edge.Cuts")
 	)
-	(gr_arc
+	(gr_line
 		(start 128.305 70)
-		(mid 129.203026 70.371974)
-		(end 129.575 71.27)
+		(end 99.095 70)
 		(stroke
 			(width 0.15)
@@
 	)
 	(gr_arc
-		(start 129.575 137.31)
-		(mid 129.203026 138.208026)
-		(end 128.305 138.58)
+		(start 128.305 70)
+		(mid 129.203026 70.371974)
+		(end 129.575 71.27)
 		(stroke
 			(width 0.15)
@@
 		(layer "Edge.Cuts")
 	)
-	(gr_line
-		(start 97.825 71.27)
-		(end 97.825 137.31)
+	(gr_arc
+		(start 129.575 137.31)
+		(mid 129.203026 138.208026)
+		(end 128.305 138.58)
 		(stroke
 			(width 0.15)
@@
 		)
 	)
-	(gr_text "Rev. 3"
+	(gr_text "Rev. 4"
 		(at 103.54 136.802 0)
 		(layer "B.SilkS")
