File: schematics/tms99105/bionic-tms99105.kicad_sch (KiCad schematic)
At the start: 8 parts, among them J1 Bionic-P135, J2 Bionic-P245, U1 TMS99105, U2 11AA010-I/TT

Commit message: [tms9900] Add automation config
The TMS9980, TMS9995, TMS99105 and TMS99110 run TMS9900 code. Fix the
TMS9980's program memory writes and the TMS9995's on-chip memory map.
Connections:
- net P36: now also J1.17 (P36); no longer J1.18 (P37)
- net P37: now also J1.18 (P37); no longer J1.17 (P36)
