File: schematics/hd6120/bionic-hd6120.kicad_pcb (KiCad board)
At the start: 2 copper layers, 25.4 x 68.6 mm, 13 parts, among them J1 Bionic-P135, J2 Bionic-P245, U1 HD6120, U2 11AA010-I/TT, U3 74LS05

Commit message: [schematics] Straighten board tracks and regenerate Gerbers
straighten_tracks.py on every routed board: router leftovers snapped to
0/45/90 degrees and redundant segments merged, each pass DRC-checked
(counts unchanged). Gerbers and drill files of the changed boards are
regenerated with each board's plot settings, keeping the committed file
sets; tms9980 keeps its tracks (the rebuild left a dangling VCC stub).
Routing:
- net Net-(J2-P57): track 4.42 -> 3.62 mm
- net /P13: track 44.3 -> 43.6 mm
- net /P46: track 24.1 -> 23.5 mm

Commit message: [schematics] Remove the JLC order-number marker from all boards
Other:
- board text removed: "JLCJLCJLCJLC"
Changed lines of the file:
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@@
-		)
-	)
-	(gr_text "JLCJLCJLCJLC"
-		(at 113.7 137.31 0)
-		(layer "B.SilkS")
-		(effects
-			(font
-				(size 0.8 0.8)
-			)
-			(justify bottom mirror)
 		)
 	)
