File: schematics/mezzanine/mezzanine.kicad_pcb (KiCad board)
At the start: 2 copper layers, 96.5 x 80 mm, 22 parts, among them J1 Bionic-P135, J10 Y0-7, J11 A0-7, J12 B0-7, J2 Bionic-P245, J3 Conn_01x24, J4 Conn_01x24, J5 P1P2, J6 P3P4, J7 P5, J8 5V0, J9 GND, U1 CPU, U2 11AA010-I/TT, U3 74AHCT157, U4 74AHCT157

Commit message: [schematics] Straighten board tracks and regenerate Gerbers
straighten_tracks.py on every routed board: router leftovers snapped to
0/45/90 degrees and redundant segments merged, each pass DRC-checked
(counts unchanged). Gerbers and drill files of the changed boards are
regenerated with each board's plot settings, keeping the committed file
sets; tms9980 keeps its tracks (the rebuild left a dangling VCC stub).
Routing:
- net /B.1: track 39.6 -> 38.7 mm

Commit message: [schematics] Align silkscreen reference labels
align_silk.py snaps each footprint kind's labels onto their common
offset and angle and clears labels DRC flags on silkscreen; 76 labels on
22 boards, no DRC count grows. Their Gerbers are regenerated.
Changed lines of the file:
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@@
 		(tags "capacitor handsolder")
 		(property "Reference" "C1"
-			(at 2.6935 0 90)
+			(at 2.74 0 90)
 			(layer "F.SilkS")
 			(effects
@@
 		(tags "capacitor handsolder")
 		(property "Reference" "C2"
-			(at 2.794 0 90)
-			(layer "F.SilkS")
-			(effects
+			(at 2.74 0 90)
+			(layer "F.SilkS")
+			(effects

Commit message: [schematics] Remove the JLC order-number marker from all boards
Other:
- board text removed: "JLCJLCJLCJLC"
Changed lines of the file:
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@@
-		)
-	)
-	(gr_text "JLCJLCJLCJLC"
-		(at 78.74 110.236 -0)
-		(layer "B.SilkS")
-		(effects
-			(font
-				(size 0.8 0.8)
-				(thickness 0.1)
-			)
-			(justify mirror)
 		)
 	)
