File: schematics/p8080/bionic-p8080.kicad_pcb (KiCad board)
At the start: 2 copper layers, 25.4 x 68.6 mm, 27 parts, among them J1 Bionic-P135, J2 Bionic-P245, Q1 2N7002DW, U1 P8080A, U2 11AA010-I/TT, U3 NJW4132, U4 NJW4191, U5 74AHCT2G126, U6 74AHCT2G126

Commit message: [schematics] Straighten board tracks and regenerate Gerbers
straighten_tracks.py on every routed board: router leftovers snapped to
0/45/90 degrees and redundant segments merged, each pass DRC-checked
(counts unchanged). Gerbers and drill files of the changed boards are
regenerated with each board's plot settings, keeping the committed file
sets; tms9980 keeps its tracks (the rebuild left a dangling VCC stub).
Routing:
- net +12V: track 50.3 -> 46.7 mm
- net /P10: track 27.4 -> 26.2 mm
- net /P23: track 27.1 -> 26.0 mm
- net /P47: track 8.55 -> 7.42 mm
- net VCC: track 156.7 -> 155.9 mm
- net /dcdc-5v/-5V: track 40.4 -> 39.7 mm
- net Net-(J2-P57): track 2.93 -> 2.29 mm
- net /P46: track 8.62 -> 8.05 mm

Commit message: [schematics] Align silkscreen reference labels
align_silk.py snaps each footprint kind's labels onto their common
offset and angle and clears labels DRC flags on silkscreen; 76 labels on
22 boards, no DRC count grows. Their Gerbers are regenerated.
Changed lines of the file:
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@@
 		(tags "capacitor handsolder")
 		(property "Reference" "C2"
-			(at -0.0011 -1.2954 90)
+			(at 0 -1.04 90)
 			(layer "F.SilkS")
 			(effects

Commit message: [schematics] Remove the JLC order-number marker from all boards
Other:
- board text removed: "JLCJLCJLCJLC"
Changed lines of the file:
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@@
-		)
-	)
-	(gr_text "JLCJLCJLCJLC"
-		(at 113.7 137.31 0)
-		(layer "B.SilkS")
-		(effects
-			(font
-				(size 0.8 0.8)
-			)
-			(justify bottom mirror)
 		)
 	)
