File: schematics/mos6502/bionic-mos6502.kicad_sch (KiCad schematic)
At the start: 8 parts, among them J1 Bionic-P135, J2 Bionic-P245, U1 W65C816S, U2 11AA010-I/TT

Commit message: [mos6502] Move PHI0 to P47 and run CMOS parts from a PWM clock (rev 11)
PHI0 on P55 has no FlexPWM output; P47 does. Rev 11 moves PHI0 there
and swaps PHI2O, E and PHI1O around it. Reset tells the parts apart
bit-banged, then the G65SC02, R65C02, W65C02S and W65C816S hand PHI0
to the PWM at a rate per part, holding each cycle with RDY; the NMOS
6502 ignores RDY on writes and stays bit-banged. Unbenched: the rev 11
board does not exist yet.
Connections:
- net P43: now also U1.35 (E); no longer U1.39 (VDA)
- net P46: now also U1.39 (VDA); no longer U1.35 (E)
- net P47: now also U1.37 (PHI2I); no longer U1.3 (~{ABORT})
- net P55: now also U1.3 (~{ABORT}); no longer U1.37 (PHI2I)
Changed lines of the file:
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@@
 	(title_block
 		(title "BionicMOS6502")
-		(date "2025-03-02")
-		(rev "10")
+		(date "2026-10-28")
+		(rev "11")
 		(company "Tadashi G. Takaoka")
 	)
@@
 	)
 	(bus_entry
-		(at 59.69 100.33)
+		(at 63.5 100.33)
 		(size -2.54 -2.54)
 		(stroke
@@
 	)
 	(bus_entry
-		(at 63.5 120.65)
+		(at 59.69 120.65)
 		(size -2.54 -2.54)
 		(stroke
@@
 	(wire
 		(pts
-			(xy 59.69 100.33) (xy 72.39 100.33)
+			(xy 63.5 100.33) (xy 72.39 100.33)
 		)
 		(stroke
@@
 	(bus
 		(pts
-			(xy 60.96 107.95) (xy 60.96 118.11)
-		)
-		(stroke
-			(width 0)
-			(type default)
-		)
-	)
-	(bus
-		(pts
 			(xy 132.08 64.77) (xy 132.08 105.41)
 		)
@@
 	(wire
 		(pts
-			(xy 63.5 120.65) (xy 72.39 120.65)
-		)
-		(stroke
-			(width 0)
-			(type default)
-		)
-	)
-	(bus
-		(pts
-			(xy 60.96 95.25) (xy 60.96 102.87)
+			(xy 59.69 120.65) (xy 72.39 120.65)
+		)
+		(stroke
+			(width 0)
+			(type default)
+		)
+	)
+	(bus
+		(pts
+			(xy 60.96 95.25) (xy 60.96 97.79)
+		)
+		(stroke
+			(width 0)
+			(type default)
+		)
+	)
+	(bus
+		(pts
+			(xy 60.96 97.79) (xy 60.96 102.87)
 		)
 		(stroke
@@
 	(bus
 		(pts
-			(xy 57.15 97.79) (xy 57.15 57.15)
+			(xy 57.15 118.11) (xy 57.15 57.15)
 		)
 		(stroke
@@
 		)
 	)
-	(label "P47"
+	(label "P55"
 		(at 71.12 100.33 180)
 		(fields_autoplaced yes)
@@
 		)
 	)
-	(label "P46"
+	(label "P43"
 		(at 96.52 115.57 0)
 		(fields_autoplaced yes)
@@
 		)
 	)
-	(label "P55"
+	(label "P47"
 		(at 71.12 120.65 180)
 		(fields_autoplaced yes)
@@
 		)
 	)
-	(label "P43"
+	(label "P46"
 		(at 96.52 125.73 0)
 		(fields_autoplaced yes)
